File: hardware/electronics/work_on_progree_pn5180_board/pn5180_board.kicad_pcb (KiCad board)
At the start: 2 copper layers, 70 x 39 mm, 73 parts, among them J1 10 pin IDC connector, Q1 AO3400A, U1 REQ, U2 PN5180, U3 TX1, U4 TX2, U5 TX_supply, U6 GND, U7 HEF4093B, U8 3.3V, U9 5V, Y1 27.12 MHz

Commit message: BOM added
Parts:
- moved RL1 0.09 mm to (151.5, 119.4)
Connections:
- C17 pad 2: Net-(U2-TVSS) -> GND
- C18 pad 1: Net-(U2-TVSS) -> GND
- C21 pad 2: Net-(U2-TVSS) -> GND
- C22 pad 1: Net-(U2-TVSS) -> GND
- C24 pad 1: Net-(U2-TVSS) -> GND
- C25 pad 2: Net-(U2-TVSS) -> GND
- C33 pad 1: Net-(U2-TVSS) -> GND
- C34 pad 2: Net-(U2-TVSS) -> GND
- C35 pad 1: Net-(U2-TVSS) -> GND
- C36 pad 2: Net-(U2-TVSS) -> GND
- C38 pad 1: Net-(U2-TVSS) -> GND
- C39 pad 2: Net-(U2-TVSS) -> GND
- U2 pad 19: Net-(U2-TVSS) -> GND
Routing:
- net GND: track 28.6 -> 73.9 mm, vias 168 -> 180
- net Net-(U2-TVSS): track 42.0 -> 0.00 mm

Commit message: pn5180 board rev 2.0
Parts:
- added C23: open, my_footprints:C_aux, F.Cu at (160.0, 112.9)
- added R14: 1Ohm, Resistor_SMD:R_0603_1608Metric, F.Cu at (140.3, 121.0)
- added R15: open, Resistor_THT:R_Axial_DIN0207_L6.3mm_D2.5mm_P10.16mm_Horizontal, F.Cu at (121.3, 108.2)
- added R16: open, Resistor_THT:R_Axial_DIN0207_L6.3mm_D2.5mm_P10.16mm_Horizontal, F.Cu at (122.5, 124.2)
- added R17: 1Ohm, Resistor_SMD:R_0603_1608Metric, F.Cu at (140.4, 109.0)
- added U13: GND, my_footprints:1pin, F.Cu at (149.1, 145.1)
- added U14: GND, my_footprints:1pin, F.Cu at (155.0, 135.0)
- C14, C15: value 1.5 pF -> 1nF
- C17, C18: value 100pF -> 56pF
- C21, C22: value 27pF -> 68pF
- C28, C31: value 15pF -> N.C.
- C29, C30: value 68pF -> 47pF
- C35, C36: value 22pF -> 68pF
- R10, R11: value 2R7 -> 2Ohm
- moved C8 1.98 mm to (125.9, 121.2), turned to 0 degrees
- moved R12 1.15 mm to (134.9, 123.4)
Routing:
- net Net-(C23-Pad2): track 13.9 -> 24.7 mm
- net Net-(C18-Pad2): track 15.1 -> 23.0 mm
- net Net-(C15-Pad2): track 1.51 -> 9.03 mm, vias 0 -> 1
- net Net-(C23-Pad1): track 7.07 -> 14.6 mm
- net Net-(C14-Pad2): track 1.51 -> 8.15 mm, vias 0 -> 1
- net Net-(C17-Pad1): track 15.2 -> 21.5 mm
- net Net-(R11-Pad1): track 20.2 -> 26.6 mm
- net Net-(R10-Pad2): track 6.68 -> 12.3 mm
- net +3.3V: track 97.3 -> 100.4 mm
- net Net-(C30-Pad2): track 17.6 -> 19.5 mm
- net Net-(C27-Pad2): track 17.6 -> 19.1 mm
- net GND: track 73.9 -> 73.8 mm, vias 180 -> 164
Other:
- board text added: "PN5180 NFC Reader V2"
- board text removed: "PN5180 NFC Reader V1"
