File: hardware/electronics/work_on_progree_pn5180_board/pn5180_board.kicad_sch (KiCad schematic)
At the start: 73 parts, among them J1 10 pin IDC connector, Q1 AO3400A, U1 REQ, U2 PN5180, U3 TX1, U4 TX2, U5 TX_supply, U6 GND, U7 HEF4093B, U8 3.3V, U9 5V, Y1 27.12 MHz

Commit message: BOM added
Parts:
- RL1: footprint Relay_THT:Relay_DPDT_Panasonic_JW2 -> my_footprints:Relay
Connections:
- net GND: now also C17.2, C18.1, C21.2, C22.1, C24.1, C25.2, C33.1, C34.2, C35.1, C36.2, C38.1, C39.2, U2.19 (TVSS)
Changed lines of the file:
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@@
 	)
 	(junction
+		(at 161.29 101.6)
+		(diameter 0)
+		(color 0 0 0 0)
+	)
+	(junction
 		(at 120.65 135.89)
 		(diameter 0)
@@
 	)
 	(junction
+		(at 119.38 101.6)
+		(diameter 0)
+		(color 0 0 0 0)
+	)
+	(junction
 		(at 69.85 127)
 		(diameter 0)
@@
 	(wire
 		(pts
+			(xy 190.5 101.6) (xy 193.04 101.6)
+		)
+		(stroke
+			(width 0)
+			(type default)
+		)
+	)
+	(wire
+		(pts
 			(xy 231.14 129.54) (xy 231.14 133.35)
 		)
@@
 	(wire
 		(pts
+			(xy 119.38 101.6) (xy 123.19 101.6)
+		)
+		(stroke
+			(width 0)
+			(type default)
+		)
+	)
+	(wire
+		(pts
 			(xy 175.26 39.37) (xy 175.26 40.64)
 		)
@@
 	(wire
 		(pts
-			(xy 106.68 101.6) (xy 123.19 101.6)
+			(xy 106.68 101.6) (xy 119.38 101.6)
 		)
 		(stroke
@@
 	(wire
 		(pts
-			(xy 147.32 101.6) (xy 170.18 101.6)
+			(xy 147.32 101.6) (xy 161.29 101.6)
 		)
 		(stroke
@@
 	(wire
 		(pts
+			(xy 161.29 101.6) (xy 170.18 101.6)
+		)
+		(stroke
+			(width 0)
+			(type default)
+		)
+	)
+	(wire
+		(pts
 			(xy 41.91 133.35) (xy 41.91 134.62)
 		)
@@
 	(symbol
 		(lib_id "power:GND")
+		(at 119.38 101.6 0)
+		(unit 1)
+		(exclude_from_sim no)
+		(in_bom yes)
+		(on_board yes)
+		(dnp no)
+		(property "Reference" "#PWR028"
+			(at 119.38 107.95 0)
+			(effects
+				(font
+					(size 1.27 1.27)
+				)
+				(hide yes)
+			)
+		)
+		(property "Value" "GND"
+			(at 116.84 102.108 90)
+			(effects
+				(font
+					(size 1.27 1.27)
+				)
+				(justify right)
+				(hide yes)
+			)
+		)
+		(property "Footprint" ""
+			(at 119.38 101.6 0)
+			(effects
+				(font
+					(size 1.27 1.27)
+				)
+				(hide yes)
+			)
+		)
+		(property "Datasheet" ""
+			(at 119.38 101.6 0)
+			(effects
+				(font
+					(size 1.27 1.27)
+				)
+				(hide yes)
+			)
+		)
+		(property "Description" "Power symbol creates a global label with name \"GND\" , ground"
+			(at 119.38 101.6 0)
+			(effects
+				(font
+					(size 1.27 1.27)
+				)
+				(hide yes)
+			)
+		)
+		(pin "1"
+		)
+		(instances
+			(project "pn5180_board"
+				(path "/00d8f431-3556-4bff-9279-20a4c885e26b"
+					(reference "#PWR028")
+					(unit 1)
+				)
+			)
+		)
+	)
+	(symbol
+		(lib_id "power:GND")
 		(at 76.2 180.34 0)
 		(unit 1)
@@
 			)
 		)
-		(property "Footprint" "Relay_THT:Relay_DPDT_Panasonic_JW2"
+		(property "Footprint" "my_footprints:Relay"
 			(at 215.9 91.44 0)
 			(effects
@@
 	)
 	(symbol
+		(lib_id "power:GND")
+		(at 193.04 101.6 90)
+		(unit 1)
+		(exclude_from_sim no)
+		(in_bom yes)
+		(on_board yes)
+		(dnp no)
+		(property "Reference" "#PWR040"
+			(at 199.39 101.6 0)
+			(effects
+				(font
+					(size 1.27 1.27)
+				)
+				(hide yes)
+			)
+		)
+		(property "Value" "GND"
+			(at 193.548 104.14 90)
+			(effects
+				(font
+					(size 1.27 1.27)
+				)
+				(justify right)
+				(hide yes)
+			)
+		)
+		(property "Footprint" ""
+			(at 193.04 101.6 0)
+			(effects
+				(font
+					(size 1.27 1.27)
+				)
+				(hide yes)
+			)
+		)
+		(property "Datasheet" ""
+			(at 193.04 101.6 0)
+			(effects
+				(font
+					(size 1.27 1.27)
+				)
+				(hide yes)
+			)
+		)
+		(property "Description" "Power symbol creates a global label with name \"GND\" , ground"
+			(at 193.04 101.6 0)
+			(effects
+				(font
+					(size 1.27 1.27)
+				)
+				(hide yes)
+			)
+		)
+		(pin "1"
+		)
+		(instances
+			(project "pn5180_board"
+				(path "/00d8f431-3556-4bff-9279-20a4c885e26b"
+					(reference "#PWR040")
+					(unit 1)
+				)
+			)
+		)
+	)
+	(symbol
 		(lib_id "power:+5V")
 		(at 231.14 118.11 270)
@@
 					(unit 1)
 				)
+			)
+		)
+	)
+	(symbol
+		(lib_id "power:GND")
+		(at 161.29 101.6 0)
+		(unit 1)
+		(exclude_from_sim no)
+		(in_bom yes)
+		(on_board yes)
+		(dnp no)
+		(property "Reference" "#PWR039"
+			(at 161.29 107.95 0)
+			(effects
+				(font
+					(size 1.27 1.27)
+				)
+				(hide yes)
+			)
+		)
+		(property "Value" "GND"
+			(at 158.75 102.108 90)
+			(effects
+				(font
+					(size 1.27 1.27)
+				)
+				(justify right)
+				(hide yes)
+			)
+		)
+		(property "Footprint" ""
+			(at 161.29 101.6 0)
+			(effects
+				(font
+					(size 1.27 1.27)
+				)
+				(hide yes)
+			)
+		)
+		(property "Datasheet" ""
+			(at 161.29 101.6 0)
+			(effects
+				(font
+					(size 1.27 1.27)
+				)
+				(hide yes)
+			)
+		)
+		(property "Description" "Power symbol creates a global label with name \"GND\" , ground"
+			(at 161.29 101.6 0)
+			(effects
+				(font
+					(size 1.27 1.27)
+				)
+				(hide yes)
+			)
+		)
+		(pin "1"
+		)
+		(instances
+			(project "pn5180_board"
+				(path "/00d8f431-3556-4bff-9279-20a4c885e26b"
+					(reference "#PWR039")
+					(unit 1)
+				)

Commit message: pn5180 board rev 2.0
Parts:
- added C23: open, my_footprints:C_aux, symbol Device:C
- added R14, R17: 1Ohm, Resistor_SMD:R_0603_1608Metric, symbol Device:R
- added R15, R16: open, Resistor_THT:R_Axial_DIN0207_L6.3mm_D2.5mm_P10.16mm_Horizontal, symbol Device:R
- added U13, U14: GND, my_footprints:1pin, symbol New_Library:1_pin
- C14, C15: value 1.5 pF -> 1nF; LCSC C1552 -> C1523
- C17, C18: value 100pF -> 56pF; LCSC C14858 -> C39148
- C21, C22: value 27pF -> 68pF; LCSC C1656 -> C28262
- C28, C31: value 15pF -> N.C.; LCSC C1644 -> (none)
- C29, C30: value 68pF -> 47pF; LCSC C28262 -> C1671
- C35, C36: value 22pF -> 68pF; LCSC C1653 -> C28262
- C38, C39: LCSC C1653 -> (none)
- R10, R11: value 2R7 -> 2Ohm; LCSC C2930033 -> C22977
Connections:
- net GND: now also U13.1 (pin), U14.1 (pin)
- net at C27.2, C28.2, C29.2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: now also R17.1
- net at R10.2, R9.2, RL1.5: now also R17.2
- net at C18.2, C22.2, C25.1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: now also R16.2
- net at C30.2, C31.2, C32.2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: now also R14.1
- net at R11.1, R12.2, RL1.4: now also R14.2
- net at C15.2, R5.1: now also R16.1
- net at C17.1, C21.1, C24.2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: now also R15.2
- net at C14.2, R4.1: now also R15.1
- net at L4.1, RL1.6: now also C23.2
- net at L4.2, RL1.3: now also C23.1
Other:
- moved on the sheet: L4, R12, R9, U7C, U7D, U7E
